Commit message: included a new laser frame link for the lidar component and also a new color mat to make it red in gazebo

File: description/lidar.xacro (robot description, xacro)
@@ -6,3 +6,19 @@
         <origin xyz="0.1 0 0.175" rpy="0 0 0"/>
     </joint>
+    <link name="laser_frame">
+        <visual>
+            <geometry>
+                <cylinder radius="0.05" length="0.04"/>
+            </geometry>
+            <material name="red"/>
+        </visual>
+        <collision>
+            <geometry>
+                <cylinder radius="0.05" length="0.04"/>
+            </geometry>
+        </collision>
+        <xacro:inertial_cylinder mass="0.1" length="0.04" radius="0.05">
+            <origin xyz="0 0 0" rpy="0 0 0"/>
+        </xacro:inertial_cylinder>
+    </link>
 </robot>

File: description/robot_core.xacro (robot description, xacro)
@@ -44,4 +44,7 @@
         <material>Gazebo/White</material>
     </gazebo>
+    <material name="red">
+        <color rgba="1 0 0 1"/>
+    </material>
     <!-- LEFT WHEEL LINK -->
     <joint name="left_wheel_joint" type="continuous">
