Commit message: moved new red mat and created a new gazebo tag that references the laser_frame

File: description/robot_core.xacro (robot description, xacro)
@@ -13,4 +13,7 @@
     <material name="black">
         <color rgba="0 0 0 1"/>
+    </material>
+    <material name="red">
+        <color rgba="1 0 0 1"/>
     </material>
     <!-- BASE LINK -->
@@ -44,7 +47,4 @@
         <material>Gazebo/White</material>
     </gazebo>
-    <material name="red">
-        <color rgba="1 0 0 1"/>
-    </material>
     <!-- LEFT WHEEL LINK -->
     <joint name="left_wheel_joint" type="continuous">
@@ -126,3 +126,6 @@
         <mu2 value="0.001"/>
     </gazebo>
+    <gazebo reference="laser_frame">
+        <material>Gazebo/Red</material>
+    </gazebo>
 </robot>
